File: Lower_Pad.kicad_sch (KiCad schematic)
At the start: 40 parts, among them SW54 INIT, SW58 SEC F-PLN, SW59 A, SW60 F, SW61 K, SW62 DATA, SW63 ATC COMM, SW64 B, SW65 G, SW66 L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

Commit message: Finished all button
Parts:
- removed D54, D58, D62, D63, D67: 1N4148, Diode_THT:D_DO-35_SOD27_P7.62mm_Horizontal, symbol Diode:1N4148
- removed SW54: INIT, 1825910_6:SW_1825910-6-4, symbol 1825910-6:1825910-6
- removed SW58: SEC F-PLN, 1825910_6:SW_1825910-6-4, symbol 1825910-6:1825910-6
- removed SW62: DATA, 1825910_6:SW_1825910-6-4, symbol 1825910-6:1825910-6
- removed SW63: ATC COMM, 1825910_6:SW_1825910-6-4, symbol 1825910-6:1825910-6
- removed SW67: MCDU MENU, 1825910_6:SW_1825910-6-4, symbol 1825910-6:1825910-6
- SW59: value A -> P
- SW60: value F -> U
- SW61: value K -> Z
- SW64: value B -> Q
- SW65: value G -> V
- SW66: value L -> /
- SW68: value C -> R
- SW69: value H -> W
- SW70: value M -> SP
- SW71: value D -> S
- SW72: value I -> X
- SW73: value N -> OVFY
- SW74: value E -> T
- SW75: value J -> Y
- SW76: value O -> CLR
Connections:
- net ROW_2 renamed ROW_5
- net ROW_3 renamed ROW_6
- net ROW_4 renamed ROW_7
- no-connect marks 40 -> 30
