File: pico.kicad_sch (KiCad schematic)
At the start: 0 parts

Commit message: Add: PCB Part, NumPad Mesurement
Parts:
- added A1: RaspberryPi_Pico, Module:RaspberryPi_Pico_Common_Unspecified, symbol MCU_Module:RaspberryPi_Pico
Connections:
- new net: A1.13 (GND), A1.18 (GND), A1.23 (GND), A1.28 (GND), A1.3 (GND), A1.38 (GND), A1.8 (GND)
- new net COL_0: A1.1 (GPIO0)
- new net COL_1: A1.2 (GPIO1)
- new net COL_2: A1.4 (GPIO2)
- new net COL_3: A1.5 (GPIO3)
- new net COL_4: A1.6 (GPIO4)
- new net COL_5: A1.7 (GPIO5)
- new net COL_6: A1.9 (GPIO6)
- new net COL_7: A1.10 (GPIO7)
- new net COL_8: A1.11 (GPIO8)
- new net ROW_0: A1.12 (GPIO9)
- new net ROW_1: A1.14 (GPIO10)
- new net ROW_2: A1.15 (GPIO11)
- new net ROW_3: A1.16 (GPIO12)
- new net ROW_4: A1.17 (GPIO13)
- new net ROW_5: A1.19 (GPIO14)
- new net ROW_6: A1.20 (GPIO15)
- new net ROW_7: A1.21 (GPIO16)
- new net ROW_8: A1.22 (GPIO17)
- no-connect marks 0 -> 16
