File: A320_MCDU.kicad_pcb (KiCad board)
At the start: 2 copper layers, 146.2 x 227.2 mm, 145 parts, among them SW1 1, SW10 ., SW11 0, SW12 +/-, SW13 DIR, SW14 F-PLN, SW15 AIR PORT, SW16 →, SW17 PROG, SW18 RAD NAV, SW19 LSK1L, SW2 2, SW20 ↓, SW21 BRT, SW22 DIM, SW23 LSK2L, SW24 LSK3L, SW25 PERF, SW26 FUEL PRED, SW27 LSK4L, SW28 LSK5L, SW29 INIT, SW3 3, SW30 SEC F-PLN, SW31 A, SW32 K, SW33 DATA, SW34 ATC COMM, SW35 B, SW36 L, SW37 LSK6L, SW38 MCDU MENU, SW39 C, SW4 4, SW40 M, SW41 ←, SW42 ↑, SW43 LSK1R, SW44 F, SW45 G, SW46 H, SW47 LSK2R, SW48 LSK3R, SW49 LSK4R, SW5 5, SW50 D, SW51 I, SW52 N, SW53 LSK5R, SW54 LSK6R, SW55 E, SW56 J, SW57 O, SW59 P, SW6 6, SW60 U, SW61 Z, SW64 Q, SW65 V, SW66 /, SW68 R, SW69 W, SW7 7, SW70 SP, SW71 S, SW72 X, SW73 OVFY, SW74 T, SW75 Y, SW76 CLR, SW8 8, SW9 9

Commit message: Add: PCB Part, Just need routage rn
Parts:
- moved SW21 543.6 mm to (443.4, 106.3), turned to 90 degrees
- moved D76 541.4 mm to (433.5, 215.5), turned to 90 degrees
- moved SW22 540.9 mm to (443.4, 119.0), turned to 90 degrees
- moved D75 540.3 mm to (433.5, 202.6), turned to 90 degrees
- moved D74 539.1 mm to (433.4, 187.7), turned to 90 degrees
- moved D73 528.0 mm to (418.5, 215.4), turned to 90 degrees
- moved SW47 527.0 mm to (454.6, 35.4)
- moved SW48 526.6 mm to (454.6, 46.7)
- moved D72 526.6 mm to (418.4, 202.4), turned to 90 degrees
- moved SW43 525.8 mm to (454.7, 24.1)
- moved D71 525.1 mm to (418.3, 187.6), turned to 90 degrees
- moved SW76 519.3 mm to (441.0, 210.1)
- moved SW75 518.0 mm to (441.0, 195.2)
- moved SW74 516.8 mm to (441.0, 180.3)
- moved SW49 515.7 mm to (454.6, 58.0)
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
Commit message: Finished: PCB
Routing:
- net /Lower Pad/COL_6: track 0.00 -> 467.0 mm, vias 0 -> 1
- net /Lower Pad/COL_5: track 0.00 -> 397.9 mm, vias 0 -> 1
- net /Pico/ROW_4: track 0.00 -> 393.6 mm, vias 0 -> 1
- net /Pico/ROW_2: track 0.00 -> 380.4 mm, vias 0 -> 3
- net /Pico/ROW_3: track 0.00 -> 378.7 mm, vias 0 -> 5
- net /Lower Pad/COL_7: track 0.00 -> 367.3 mm, vias 0 -> 1
- net /NumPad/COL_2: track 0.00 -> 355.1 mm
- net /Pico/ROW_0: track 0.00 -> 338.6 mm, vias 0 -> 1
- net /Lower Pad/ROW_7: track 0.00 -> 317.8 mm, vias 0 -> 1
- net /Pico/COL_8: track 0.00 -> 315.0 mm
- net /NumPad/ROW_8: track 0.00 -> 314.5 mm, vias 0 -> 1
- net /NumPad/COL_1: track 0.00 -> 310.7 mm
- net /Pico/ROW_1: track 0.00 -> 305.4 mm, vias 0 -> 1
- net /Lower Pad/COL_4: track 0.00 -> 284.9 mm
- net /Lower Pad/ROW_6: track 0.00 -> 278.1 mm
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